File: XICIE_AFE/afe_revC.sch (EAGLE design)
At the start: 26 parts, among them IC1 LM324N, T1 SFH303

Commit message: Minor changes in AFE revC and added DISPLAY board
Parts:
- removed C10, C9: 0.22u, rcl:C-EU102-043X133
- removed C8: 0.1u, rcl:C-EU050-024X044
- removed R10: 33K, rcl:R-US_0207/10
- removed R11: 3.3K, rcl:R-US_0207/10
- added R1: 150K, rcl:R-US_0207/10
- R9: value 33K -> 150K
Connections:
- removed net N$10: C10.1, C9.2, R11.2
- removed net N$11: IC1D.-IN, IC1D.OUT, LED2.A
- removed net N$8: C8.2, R10.1, R9.2
- removed net N$9: C10.2, C5.+, R10.2
- new net N$15: IC1C.OUT, LED1.A
- new net N$16: IC1D.OUT, LED2.A
- net +5V: now also R9.2, T1.E
- net GND: now also R1.1; no longer T1.E
- net N$12: now also IC1D.-IN, R1.2, R9.1; no longer IC1C.OUT, LED1.A
- net N$3: now also C5.+; no longer C9.1, R9.1
- net VREF: no longer C8.1, R11.1
Other:
- moved on the sheet: IC1C, JP1, LED1, R12, R9
