File: XICIE_AFE_SMD/XICIE_AFE_SMD_revA.brd (EAGLE design)
At the start: 34 x 18 mm, 21 parts, among them IC1 LM324D, IC2 CY8C4245T, IC3 AAT1217, J1 22-27-2021-02, Q1 MOSFET-NCHANNELBSS123LT1G, Q2 MOSFET-NCHANNELBSS123LT1G

Commit message: Trying to merge display
Parts:
- removed R8: 1.02 M, rcl:R0805
- removed R9: 604 K, rcl:R0603
- added C4, C5, C6, C7: 1 uF, rcl:C0402
- added C8: 2.2 uF, rcl:C0603
- added C9: 4.7 uF, rcl:C0603
- added R5: 390K, resistor:R0603
- added U$2: ER-OLED0.96, juliano:FLEX0.7X30
Connections:
- removed net N$14: IC3.3, R8.2, R9.1
- new net C1N: C4.1, U$2.P5
- new net C1P: C4.2, U$2.P4
- new net C2N: C5.1, U$2.P3
- new net C2P: C5.2, U$2.P2
- new net CS#: U$2.P13
- new net D/C#: U$2.P15
- new net D0: U$2.P18
- new net D1: U$2.P19
- new net D2: U$2.P20
- new net D3: U$2.P21
- new net D4: U$2.P22
- new net D5: U$2.P23
- new net D6: U$2.P24
- new net D7: U$2.P25
- new net E/RD#: U$2.P17
- new net IREF: R5.1, U$2.P26
- new net N.C.: U$2.P7
- new net R/W#: U$2.P16
- new net RES#: U$2.P14
- new net V+: C6.1, U$2.P6
- new net V2.1: C9.1, U$2.P27
- new net VCC_DISPLAY: C8.1, U$2.P28
- new net VDD: C7.1, U$2.P11, U$2.P9
- net GND: now also C6.2, C7.2, C8.2, C9.2, R5.2, U$2.P1, U$2.P10, U$2.P12, U$2.P29, U$2.P30, U$2.P8; no longer R9.2
- net VCC: no longer R8.1
Routing:
- net N$14: track 5.02 -> 0.00 mm, vias 1 -> 0
- net VCC: track 16.7 -> 16.2 mm
Changed lines of the file:
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@@
 <element name="C1" library="rcl" package="C0603" value="4.7 uF" x="35.49" y="59.9"/>
 <element name="L1" library="juliano" package="L2518" value="4.7 uH" x="39.34" y="64.6" rot="R180"/>
-<element name="R8" library="rcl" package="R0805" value="1.02 M" x="39.28" y="56.52" rot="MR0"/>
-<element name="R9" library="rcl" package="R0603" value="604 K" x="34.98" y="57.94" rot="MR0"/>
 <element name="C3" library="rcl" package="C0603" value="4.7 uF" x="39.42" y="56.79" rot="R180"/>
 <element name="D1" library="juliano" package="SMINI2-F5-B" value="" x="39.05" y="62.44" rot="R180"/>
@@
 <attribute name="VALUE" x="38.4631" y="67.3989" size="0.8128" layer="27" ratio="10" rot="R180"/>
 </element>
+<element name="C4" library="rcl" package="C0402" value="1 uF" x="23.65" y="26.75"/>
+<element name="C5" library="rcl" package="C0402" value="1 uF" x="28.6" y="26.75"/>
+<element name="C6" library="rcl" package="C0402" value="1 uF" x="33.55" y="26.75"/>
+<element name="C7" library="rcl" package="C0402" value="1 uF" x="38.5" y="26.75"/>
+<element name="C8" library="rcl" package="C0603" value="2.2 uF" x="28.95" y="31.9"/>
+<element name="C9" library="rcl" package="C0603" value="4.7 uF" x="35.4" y="31.9"/>
+<element name="R5" library="resistor" package="R0603" value="390K" x="23.65" y="31.65"/>
+<element name="U$2" library="juliano" package="FLEX0.7X30" value="ER-OLED0.96" x="33.2" y="37.2"/>
 </elements>
 <signals>
@@
 <contactref element="IC2" pad="35"/>
 <contactref element="C3" pad="1"/>
-<contactref element="R8" pad="1"/>
 <contactref element="IC3" pad="5"/>
 <contactref element="D1" pad="C"/>
@@
 <wire x1="40" y1="58" x2="40" y2="57" width="0.254" layer="16"/>
 <wire x1="40" y1="57" x2="40" y2="58" width="0.254" layer="1"/>
-<wire x1="40" y1="57" x2="40.23" y2="56.52" width="0.254" layer="16"/>
 <wire x1="40" y1="57" x2="40.27" y2="56.79" width="0.254" layer="1"/>
 <via x="40" y="58" extent="1-16" drill="0.3302"/>
@@
 <wire x1="56.5" y1="62.58" x2="56.5" y2="61.45" width="0.254" layer="1"/>
 <wire x1="56.5" y1="61.45" x2="56.7" y2="60.38" width="0.254" layer="1"/>
+<wire x1="52.5" y1="64.5" x2="55.99" y2="62.58" width="0" layer="19" extent="1-16"/>
+<wire x1="44.95" y1="61.3" x2="45.780996875" y2="60.8998375" width="0" layer="19" extent="1-1"/>
+<wire x1="45.48" y1="57.75" x2="45.780996875" y2="60.8998375" width="0" layer="19" extent="1-1"/>
+<wire x1="40.71" y1="59.84" x2="44.95" y2="61.3" width="0" layer="19" extent="1-1"/>
+<wire x1="40" y1="58" x2="40.71" y2="59.84" width="0" layer="19" extent="1-16"/>
+<wire x1="40.25" y1="62.44" x2="40.71" y2="59.84" width="0" layer="19" extent="1-1"/>
 </signal>
 <signal name="GND" class="1">
@@
 <contactref element="IC3" pad="2"/>
 <contactref element="C1" pad="2"/>
-<contactref element="R9" pad="2"/>
 <contactref element="C3" pad="2"/>
 <polygon width="0.254" layer="16" rank="6">
@@
 <wire x1="54" y1="64.5" x2="53.5" y2="65" width="0.254" layer="16"/>
 <wire x1="53.5" y1="65.5" x2="53.51" y2="65.75" width="0.254" layer="16"/>
+<contactref element="U$2" pad="P10"/>
+<contactref element="U$2" pad="P12"/>
+<contactref element="U$2" pad="P1"/>
+<contactref element="C9" pad="2"/>
+<contactref element="R5" pad="2"/>
+<contactref element="C6" pad="2"/>
+<contactref element="C8" pad="2"/>
+<contactref element="C7" pad="2"/>
+<contactref element="U$2" pad="P8"/>
+<contactref element="U$2" pad="P29"/>
+<contactref element="U$2" pad="P30"/>
+<wire x1="61.71" y1="56.75" x2="61.71" y2="63.95" width="0" layer="19" extent="16-16"/>
+<wire x1="56.7" y1="55.18" x2="61.71" y2="56.75" width="0" layer="19" extent="1-16"/>
+<wire x1="54" y1="64.5" x2="61.71" y2="63.95" width="0" layer="19" extent="16-16"/>
+<wire x1="50.9" y1="63" x2="53.5" y2="65" width="0" layer="19" extent="1-16"/>
+<wire x1="49.26" y1="63.21" x2="50.9" y2="63" width="0" layer="19" extent="1-1"/>
+<wire x1="48.08" y1="54.7" x2="49.26" y2="63.21" width="0" layer="19" extent="1-1"/>
+<wire x1="38.57" y1="56.79" x2="48.08" y2="54.7" width="0" layer="19" extent="1-1"/>
+<wire x1="38.41" y1="59.84" x2="38.57" y2="56.79" width="0" layer="19" extent="1-1"/>
+<wire x1="36.34" y1="59.9" x2="38.41" y2="59.84" width="0" layer="19" extent="1-1"/>
+<wire x1="32.98" y1="63.45" x2="36.34" y2="59.9" width="0" layer="19" extent="1-1"/>
+<wire x1="43.35" y1="37.2" x2="48.08" y2="54.7" width="0" layer="19" extent="1-1"/>
+<wire x1="42.65" y1="37.2" x2="43.35" y2="37.2" width="0" layer="19" extent="1-1"/>
+<wire x1="36.25" y1="31.9" x2="42.65" y2="37.2" width="0" layer="19" extent="1-1"/>
+<wire x1="34.2" y1="26.75" x2="36.25" y2="31.9" width="0" layer="19" extent="1-1"/>
+<wire x1="39.15" y1="26.75" x2="34.2" y2="26.75" width="0" layer="19" extent="1-1"/>
+<wire x1="29.8" y1="31.9" x2="36.25" y2="31.9" width="0" layer="19" extent="1-1"/>
+<wire x1="29.35" y1="37.2" x2="29.8" y2="31.9" width="0" layer="19" extent="1-1"/>
+<wire x1="30.75" y1="37.2" x2="29.35" y2="37.2" width="0" layer="19" extent="1-1"/>
+<wire x1="27.95" y1="37.2" x2="29.35" y2="37.2" width="0" layer="19" extent="1-1"/>
+<wire x1="23.05" y1="37.2" x2="27.95" y2="37.2" width="0" layer="19" extent="1-1"/>
+<wire x1="24.5" y1="31.65" x2="29.8" y2="31.9" width="0" layer="19" extent="1-1"/>
 </signal>
 <signal name="SENSOROUT">
@@
 <vertex x="39" y="60.5"/>
 </polygon>
-</signal>
-<signal name="N$14">
-<contactref element="R8" pad="2"/>
-<contactref element="R9" pad="1"/>
-<contactref element="IC3" pad="3"/>
-<wire x1="37" y1="58" x2="38" y2="59" width="0.254" layer="1"/>
-<wire x1="36" y1="58" x2="37" y2="58" width="0.254" layer="16"/>
-<wire x1="38" y1="59" x2="38.41" y2="58.89" width="0.254" layer="1"/>
-<wire x1="36" y1="58" x2="35.83" y2="57.94" width="0.254" layer="16"/>
-<wire x1="37" y1="58" x2="38" y2="57" width="0.254" layer="16"/>
-<wire x1="38" y1="57" x2="38.33" y2="56.52" width="0.254" layer="16"/>
-<via x="37" y="58" extent="1-16" drill="0.3302"/>
 </signal>
 <signal name="SHUTDOWN">
@@
 <wire x1="56" y1="65.85" x2="57.4" y2="65.85" width="0.6096" layer="1"/>
 </signal>
+<signal name="IREF">
+<contactref element="U$2" pad="P26"/>
+<contactref element="R5" pad="1"/>
+<wire x1="22.8" y1="31.65" x2="40.55" y2="37.2" width="0" layer="19" extent="1-1"/>
+</signal>
+<signal name="D7">
+<contactref element="U$2" pad="P25"/>
+</signal>
+<signal name="D6">
+<contactref element="U$2" pad="P24"/>
+</signal>
+<signal name="D5">
+<contactref element="U$2" pad="P23"/>
+</signal>
+<signal name="D4">
+<contactref element="U$2" pad="P22"/>
+</signal>
+<signal name="D3">
+<contactref element="U$2" pad="P21"/>
+</signal>
+<signal name="D2">
+<contactref element="U$2" pad="P20"/>
+</signal>
+<signal name="D1">
+<contactref element="U$2" pad="P19"/>
+</signal>
+<signal name="D0">
+<contactref element="U$2" pad="P18"/>
+</signal>
+<signal name="E/RD#">
+<contactref element="U$2" pad="P17"/>
+</signal>
+<signal name="R/W#">
+<contactref element="U$2" pad="P16"/>
+</signal>
+<signal name="D/C#">
+<contactref element="U$2" pad="P15"/>
+</signal>
+<signal name="RES#">
+<contactref element="U$2" pad="P14"/>
+</signal>
+<signal name="CS#">
+<contactref element="U$2" pad="P13"/>
+</signal>
+<signal name="C2P">
+<contactref element="C5" pad="2"/>
+<contactref element="U$2" pad="P2"/>
+<wire x1="29.25" y1="26.75" x2="23.75" y2="37.2" width="0" layer="19" extent="1-1"/>
+</signal>
+<signal name="C2N">
+<contactref element="C5" pad="1"/>
+<contactref element="U$2" pad="P3"/>
+<wire x1="27.95" y1="26.75" x2="24.45" y2="37.2" width="0" layer="19" extent="1-1"/>
+</signal>
+<signal name="C1P">
+<contactref element="C4" pad="2"/>
+<contactref element="U$2" pad="P4"/>
+<wire x1="24.3" y1="26.75" x2="25.15" y2="37.2" width="0" layer="19" extent="1-1"/>
+</signal>
+<signal name="C1N">
+<contactref element="C4" pad="1"/>
+<contactref element="U$2" pad="P5"/>
+<wire x1="23" y1="26.75" x2="25.85" y2="37.2" width="0" layer="19" extent="1-1"/>
+</signal>
+<signal name="N.C.">
+<contactref element="U$2" pad="P7"/>
+</signal>
+<signal name="VDD" class="2">
+<contactref element="C7" pad="1"/>
+<contactref element="U$2" pad="P9"/>
+<contactref element="U$2" pad="P11"/>
+<wire x1="30.05" y1="37.2" x2="28.65" y2="37.2" width="0" layer="19" extent="1-1"/>
+<wire x1="37.85" y1="26.75" x2="30.05" y2="37.2" width="0" layer="19" extent="1-1"/>
+</signal>
+<signal name="V+" class="2">
+<contactref element="C6" pad="1"/>
+<contactref element="U$2" pad="P6"/>
+<wire x1="32.9" y1="26.75" x2="26.55" y2="37.2" width="0" layer="19" extent="1-1"/>
+</signal>
+<signal name="V2.1">
+<contactref element="C9" pad="1"/>
+<contactref element="U$2" pad="P27"/>
+<wire x1="34.55" y1="31.9" x2="41.25" y2="37.2" width="0" layer="19" extent="1-1"/>
+</signal>
+<signal name="VCC_DISPLAY" class="2">
+<contactref element="C8" pad="1"/>
+<contactref element="U$2" pad="P28"/>
+<wire x1="28.1" y1="31.9" x2="41.95" y2="37.2" width="0" layer="19" extent="1-1"/>
+</signal>
 </signals>

Commit message: Intermediate commit to change computers...
Parts:
- added R7: 1.02 M, rcl:R0805
- added R8: 604 k, rcl:R0603
- added R9: 150 k, rcl:R0603
- added U$3: AAT3221, juliano:SOT23-5
- added U$4: MMA7660FC, juliano:DFN10
- moved C7 35.7 mm to (20.6, 57.7), turned to 90 degrees
- moved C9 35.1 mm to (21.0, 63.9)
- moved R5 34.9 mm to (16.8, 65.8)
- moved C8 31.1 mm to (18.1, 61.0), turned to 180 degrees
- moved C4 26.2 mm to (29.1, 52.4), turned to 270 degrees
- moved C5 24.8 mm to (23.4, 51.0), turned to 270 degrees
- moved U$2 23.7 mm to (26.0, 59.8), flipped to the bottom, turned to 90 degrees
- moved C6 21.7 mm to (40.8, 47.2)
Connections:
- removed net D0: U$2.P18
- removed net D1: U$2.P19
- removed net D2: U$2.P20
- removed net V+: C6.1, U$2.P6
- removed net VDD: C7.1, U$2.P11, U$2.P9
- new net +3V3: C3.1, C6.1, D1.C, IC1.4, IC2.35, IC3.5, R2.2, R3.2, R7.1, R9.1, U$1.CATHODE1, U$1.CATHODE2, U$2.P6, U$3.1, U$4.P3
- new net N$12: IC3.3, R7.2, R8.1
- new net N$14: R9.2, U$3.3
- new net SCL: U$2.P18, U$4.P6
- new net SDA: U$2.P19, U$2.P20, U$4.P7
- net GND: now also R8.2, U$3.2, U$4.P1, U$4.P4, U$4.P8
- net VCC: now also C7.1, IC2.19, IC2.33, IC2.34, U$2.P11, U$2.P9, U$3.5, U$4.P9; no longer C3.1, D1.C, IC1.4, IC2.35, IC3.5, R2.2, R3.2, U$1.CATHODE1, U$1.CATHODE2
Routing:
- net VREF: track 24.1 -> 0.00 mm, vias 1 -> 0
- net VCC: track 16.2 -> 0.00 mm, vias 2 -> 0
- net N$4: track 14.4 -> 0.00 mm
- net IR: track 10.1 -> 0.00 mm, vias 1 -> 0
- net N$3: track 9.07 -> 0.00 mm
- net N$1: track 8.21 -> 0.00 mm
- net SENSOROUT: track 8.19 -> 0.00 mm, vias 1 -> 0
- net N$9: track 7.82 -> 0.00 mm
- net R: track 7.13 -> 0.00 mm, vias 1 -> 0
- net PWM_VREF: track 3.73 -> 0.00 mm, vias 1 -> 0
- net VBAT: track 3.27 -> 0.00 mm
- net N$7: track 2.82 -> 0.00 mm
- net N$5: track 2.61 -> 0.00 mm
- net N$6: track 2.56 -> 0.00 mm
- net N$8: track 2.14 -> 0.00 mm
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- added copper zone on layer 1, net +3V3
- removed copper zone on layer 1, net VCC
Other:
- board size 34 x 18 mm -> 101 x 60.4 mm
